File: hardware/teensy-load.kicad_pcb (KiCad board)
At the start: 2 copper layers, 33 x 67.9 mm, 27 parts, among them J101 Conn_01x02, J201 Conn_01x01_Male, Q201 BTS141, U101 TEENSY_4.0, U102 TLV4333, U201 DAC6571, U301 DAC6571

Commit message: WIP
Parts:
- added REF**: MountingHole_3mm, MountingHole:MountingHole_3mm, F.Cu at (142.9, 105.4)
- added REF**: MountingHole_3mm, MountingHole:MountingHole_3mm, F.Cu at (113.7, 105.4)
- added REF**: MountingHole_3mm, MountingHole:MountingHole_3mm, F.Cu at (128.3, 48.9)
- R206, R207, R305: moved to B.Cu
- moved R303 28.3 mm to (142.7, 95.1), turned to 0 degrees
- moved R207 28.0 mm to (141.2, 70.2), turned to 270 degrees
- moved R208 27.6 mm to (138.7, 70.2), turned to 90 degrees
- moved R206 25.1 mm to (138.7, 70.2), turned to 270 degrees
- moved R302 22.5 mm to (138.5, 95.1), turned to 0 degrees
- moved R308 17.9 mm to (125.1, 66.0), turned to 270 degrees
- moved C301 17.1 mm to (135.1, 91.3), turned to 90 degrees
- moved R301 16.1 mm to (133.9, 95.1), turned to 0 degrees
- moved R307 16.0 mm to (125.1, 62.2), turned to 270 degrees
- moved U301 14.9 mm to (133.5, 90.6), turned to 90 degrees
- moved C101 12.5 mm to (141.9, 77.5), turned to 180 degrees
- moved U102 10.2 mm to (140.5, 77.7), turned to 180 degrees
- moved R304 8.94 mm to (132.1, 77.5), turned to 180 degrees
- moved R203 8.53 mm to (127.5, 95.5), turned to 270 degrees
- moved R305 8.30 mm to (132.1, 77.5), turned to 0 degrees
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Routing:
- net /Current control/IN+: track 48.9 -> 25.4 mm
- net Net-(R301-Pad2): track 59.0 -> 36.7 mm, vias 4 -> 2
- net Net-(R204-Pad2): track 29.7 -> 44.2 mm
- net /Current control/I_SENSE: track 23.5 -> 37.4 mm, vias 1 -> 0
- net Net-(D301-Pad2): track 36.2 -> 23.7 mm, vias 2 -> 0
- net /Voltage control/V_SENSE: track 14.0 -> 24.2 mm, vias 1 -> 0
- net Net-(R307-Pad2): track 22.3 -> 30.6 mm, vias 0 -> 2
- net GND: track 42.1 -> 33.9 mm, vias 9 -> 8
- net Net-(R206-Pad1): track 11.9 -> 19.9 mm, vias 0 -> 1
- net Net-(R201-Pad1): track 28.8 -> 36.5 mm, vias 0 -> 2
- net Net-(Q201-Pad3): track 43.4 -> 35.8 mm
- net +3V3: track 12.1 -> 8.40 mm
- net /Current control/I2C_SCL: track 18.6 -> 15.9 mm, vias 1 -> 0
- net /Current control/FET_GATE: track 8.16 -> 8.78 mm
- net /Current control/I2C_SDA: track 15.3 -> 15.7 mm, vias 0 -> 2
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Other:
- board size 33 x 67.9 mm -> 36.8 x 64.1 mm
- board text added: "Teensy Load V0.1 2020-04-23"
- board text removed: "Teensy Load V0.1 2020-04-22"

Commit message: V0.1 layout for manufacture
Routing:
- net /Current control/IN+: track 25.4 -> 24.2 mm
