File: hardware/teensy-load.kicad_pcb (KiCad board)
At the start: 2 copper layers, 36.8 x 64.1 mm, 30 parts, among them J101 Conn_01x02, J201 Conn_01x01_Male, Q201 BTS141, U101 TEENSY_4.0, U102 TLV4333, U201 DAC6571, U301 DAC6571

Commit message: Start of revision 2 design changes
Parts:
- removed C101: 0.1U, Capacitor_SMD:C_0805_2012Metric_Pad1.15x1.40mm_HandSolder
- removed J201: Conn_01x01_Male, teensy-load:HeatSink_RA_T2X_64E
- removed the REF** at (128.3, 48.9)
- removed U102: TLV4333, Package_SO:SOIC-14_3.9x8.7mm_P1.27mm
- added C202: 0.1U, Capacitor_SMD:C_0805_2012Metric_Pad1.15x1.40mm_HandSolder, F.Cu at (165.8, 63.7)
- added C203: 0.1U, Capacitor_SMD:C_0805_2012Metric_Pad1.15x1.40mm_HandSolder, F.Cu at (171.8, 63.8)
- added C302: 0.1U, Capacitor_SMD:C_0805_2012Metric_Pad1.15x1.40mm_HandSolder, F.Cu at (167.2, 82.7)
- added C303: 0.1U, Capacitor_SMD:C_0805_2012Metric_Pad1.15x1.40mm_HandSolder, F.Cu at (172.0, 82.9)
- added HS201: Heatsink, teensy-load:HeatSink_RA_T2X_64E, F.Cu at (128.3, 54.3)
- added U202: TLV333IDBVR, Package_TO_SOT_SMD:SOT-23-5, F.Cu at (166.0, 69.5)
- added U203: TLV333IDBVR, Package_TO_SOT_SMD:SOT-23-5, F.Cu at (171.8, 69.6)
- added U302: LMV331, Package_TO_SOT_SMD:SOT-23-5, F.Cu at (166.9, 78.2)
- added U303: TLV333IDBVR, Package_TO_SOT_SMD:SOT-23-5, F.Cu at (171.8, 78.2)
- C301: moved to F.Cu
- moved C301 15.4 mm to (150.5, 90.6), turned to 0 degrees
- moved D301 0.12 mm to (118.8, 62.8), turned to 90 degrees
Connections:
- D301 pad 1: /Current control/FET_GATE -> Net-(D301-Pad1)
- D301 pad 2: Net-(D301-Pad2) -> /Current control/FET_GATE
Routing:
- net Net-(R204-Pad2): track 44.2 -> 0.00 mm
- net /Current control/I_SENSE: track 37.4 -> 0.63 mm
- net Net-(R301-Pad2): track 36.7 -> 2.64 mm, vias 2 -> 0
- net Net-(R201-Pad1): track 36.5 -> 6.04 mm, vias 2 -> 0
- net Net-(Q201-Pad3): track 35.8 -> 6.26 mm
- net Net-(R307-Pad2): track 30.6 -> 1.76 mm, vias 2 -> 0
- net Net-(D301-Pad2): track 23.7 -> 0.00 mm
- net Net-(R206-Pad1): track 19.9 -> 7.30 mm
- net /Voltage control/V_SENSE: track 24.2 -> 16.3 mm
- net Net-(R304-Pad1): track 7.53 -> 2.54 mm
- net +3V3: track 8.40 -> 5.31 mm, vias 3 -> 2
- net GND: track 33.6 -> 32.2 mm, vias 8 -> 7
