File: hardware/teensy-load.sch (KiCad schematic (older format))
At the start: 4 parts, among them J101 Conn_01x02, U101 TEENSY_4.0, U102 TLV4333

Commit message: After footprint check, before layout
Parts:
- C101: MPN (none) -> 885012207098
- U101: MPN (none) -> TEENSY 4.0
Changed lines of the file:
@@
 F 1 "0.1U" H 9090 5055 50  0000 L CNN
 F 2 "Capacitor_SMD:C_0805_2012Metric_Pad1.15x1.40mm_HandSolder" H 9013 4950 50  0001 C CNN
-F 3 "~" H 8975 5100 50  0001 C CNN
+F 3 "https://www.mouser.at/datasheet/2/445/885012207098-1727748.pdf" H 8975 5100 50  0001 C CNN
+F 4 "885012207098" H 8975 5100 50  0001 C CNN "MPN"
 	1    8975 5100
 	1    0    0    -1
@@
 F 1 "TEENSY_4.0" H 3650 4874 50  0000 C CNN
 F 2 "teensy-load:TEENSY_4.0" H 3650 4000 50  0001 C CNN
-F 3 "" H 3650 4000 50  0001 C CNN
+F 3 "https://www.pjrc.com/store/teensy40.html" H 3650 4000 50  0001 C CNN
+F 4 "TEENSY 4.0" H 3650 4000 50  0001 C CNN "MPN"
 	1    3650 4000
 	1    0    0    -1

Commit message: Start of revision 2 design changes
Parts:
- removed C101: 0.1U, Capacitor_SMD:C_0805_2012Metric_Pad1.15x1.40mm_HandSolder, symbol Device:C
- removed U102: TLV4333, Package_SO:SOIC-14_3.9x8.7mm_P1.27mm, symbol teensy-load:TLV4333
Other:
- note removed: "Op amp power"
Changed lines of the file:
@@
 $EndDescr
-$Comp
-L power:GND #PWR0108
-U 1 1 5E58A69A
-P 9325 5400
-F 0 "#PWR0108" H 9325 5150 50  0001 C CNN
-F 1 "GND" H 9330 5227 50  0000 C CNN
-F 2 "" H 9325 5400 50  0001 C CNN
-F 3 "" H 9325 5400 50  0001 C CNN
-	1    9325 5400
-	1    0    0    -1
-$EndComp
 $Comp
 L Connector_Generic:Conn_01x02 J101
@@
 	1    0    0    -1
 $EndComp
-$Comp
-L Device:C C101
-U 1 1 5E5D75E8
-P 8975 5100
-F 0 "C101" H 9090 5146 50  0000 L CNN
-F 1 "0.1U" H 9090 5055 50  0000 L CNN
-F 2 "Capacitor_SMD:C_0805_2012Metric_Pad1.15x1.40mm_HandSolder" H 9013 4950 50  0001 C CNN
-F 3 "https://www.mouser.at/datasheet/2/445/885012207098-1727748.pdf" H 8975 5100 50  0001 C CNN
-F 4 "885012207098" H 8975 5100 50  0001 C CNN "MPN"
-	1    8975 5100
-	1    0    0    -1
-$EndComp
-Wire Wire Line
-	9325 4975 9450 4975
-Wire Wire Line
-	9450 5175 9325 5175
-Wire Wire Line
-	8975 4950 8975 4850
-Wire Wire Line
-	8975 5250 8975 5325
 Text Notes 1700 2425 0    50   ~ 0
 IDEAS\n\n - Power from Teensy\n - Expose current and voltage for measurement by Teensy ADCs\n - Program current and maximum voltage from Teensy using I2C DACs\n\nUSE CASES\n\n - Single measurements\n - Scan programming voltage, record test item voltage and current to give V/I curve\n - Fix programming voltage, record current and test item voltage over time\n\nLIMITATIONS\n\n - Current 0 - 10A (full range of current setting DAC)\n - Max. voltage 0 - 20V (full range of max. voltage setting DAC)\n - Max. power 0 - 20W (limit by firmware)
@@
 	8225 3650 8075 3650
 $Comp
-L power:+3.3V #PWR0107
-U 1 1 5E5F5427
-P 9325 4800
-F 0 "#PWR0107" H 9325 4650 50  0001 C CNN
-F 1 "+3.3V" H 9340 4973 50  0000 C CNN
-F 2 "" H 9325 4800 50  0001 C CNN
-F 3 "" H 9325 4800 50  0001 C CNN
-	1    9325 4800
-	1    0    0    -1
-$EndComp
-$Comp
 L teensy-load:TEENSY_4.0 U101
 U 1 1 5E5F881B
@@
 	5850 4675 5850 4100
 Connection ~ 5850 4100
-Text Notes 9050 4475 0    50   ~ 0
-Op amp power
 Wire Wire Line
 	7550 4575 7975 4575
@@
 F7 "V_SENSE" O L 6600 4825 50
 $EndSheet
-Wire Wire Line
-	9325 4800 9325 4850
-Wire Wire Line
-	9325 5175 9325 5325
-Wire Wire Line
-	8975 4850 9325 4850
-Connection ~ 9325 4850
-Wire Wire Line
-	9325 4850 9325 4975
-Wire Wire Line
-	8975 5325 9325 5325
-Connection ~ 9325 5325
-Wire Wire Line
-	9325 5325 9325 5400
 Text Notes 8375 3450 0    50   ~ 0
 Device under test\nconnects here
 Text Notes 4100 5275 0    50   ~ 0
 Input impedance of Teensy ADC inputs is\nca. 7kΩ, giving an input current of about\n0.5mA on each of the two inputs used.\n(Signals going to these have op amp\ndrivers to buffer them.)
-$Comp
-L teensy-load:TLV4333 U102
-U 5 1 5E6376FF
-P 9650 5075
-F 0 "U102" H 9778 5129 50  0000 L CNN
-F 1 "TLV4333" H 9778 5038 50  0000 L CNN
-F 2 "Package_SO:SOIC-14_3.9x8.7mm_P1.27mm" H 9650 5100 50  0001 C CNN
-F 3 "http://www.ti.com/general/docs/suppproductinfo.tsp?distId=26&gotoUrl=http%3A%2F%2Fwww.ti.com%2Flit%2Fgpn%2Ftlv4333" H 9650 5100 50  0001 C CNN
-F 4 "TLV4333IDR" H 9650 5075 50  0001 C CNN "MPN"
-	5    9650 5075
-	1    0    0    -1
-$EndComp
 Text Notes 1450 6200 0    50   ~ 10
 POWER
