File: hardware/voltage-control.sch (KiCad schematic (older format))
At the start: 8 parts, among them U102 TLV4333, U301 DAC6571

Commit message: After footprint check, before layout
Parts:
- added R303, R305: 33K, Resistor_SMD:R_0805_2012Metric_Pad1.15x1.40mm_HandSolder, symbol Device:R
- added R304: 27K, Resistor_SMD:R_0805_2012Metric_Pad1.15x1.40mm_HandSolder, symbol Device:R
- added R306: 39K, Resistor_SMD:R_0805_2012Metric_Pad1.15x1.40mm_HandSolder, symbol Device:R
- C301: MPN (none) -> 885012207098
- R301: value 10K -> 39K; MPN (none) -> CRCW040239K0FKEDC
- R302: value 15K -> 27K; MPN (none) -> CRCW120627K0FKEAC
- R307: renamed from R303; value 9K -> 18K; MPN (none) -> CRGP0805F18K
- R308: renamed from R304; value 1K -> 2K; MPN (none) -> CRCW08052K00FKEAC
Connections:
- net GND: now also R303.2, R305.2; no longer R302.2
- net V_SENSE: now also R306.2; no longer U102.13 (-)
- new net: R302.2, R303.1
- new net: R304.1, R306.1, U102.13 (-)
- new net: R304.2, R305.1
Other:
- note added: "Amplification of 1.65 here gives full range\nADC input for sense voltage range of 0-2V."
- moved on the sheet: R307, R308
Changed lines of the file:
@@
 L power:GND #PWR?
 U 1 1 5E6085EF
-P 5200 4125
+P 5200 4400
 AR Path="/5E6085EF" Ref="#PWR?"  Part="1"
 AR Path="/5E5EBC79/5E6085EF" Ref="#PWR?"  Part="1"
 AR Path="/5E5EBE75/5E6085EF" Ref="#PWR0304"  Part="1"
-F 0 "#PWR0304" H 5200 3875 50  0001 C CNN
-F 1 "GND" H 5205 3952 50  0000 C CNN
-F 2 "" H 5200 4125 50  0001 C CNN
-F 3 "" H 5200 4125 50  0001 C CNN
-	1    5200 4125
+F 0 "#PWR0304" H 5200 4150 50  0001 C CNN
+F 1 "GND" H 5205 4227 50  0000 C CNN
+F 2 "" H 5200 4400 50  0001 C CNN
+F 3 "" H 5200 4400 50  0001 C CNN
+	1    5200 4400
 	1    0    0    -1
 $EndComp
@@
 Wire Wire Line
 	5200 2750 4725 2750
-Wire Wire Line
-	5200 3900 5200 4025
 Text Notes 4925 2725 0    50   ~ 0
 0-3.3V
 Text Notes 5425 3450 0    50   ~ 0
 0-2V
-Wire Wire Line
-	4275 4025 5200 4025
-Connection ~ 5200 4025
-Wire Wire Line
-	5200 4025 5200 4125
 Text Notes 3050 3100 0    50   ~ 0
 Other DAC6571\nhas A0 low
-Wire Wire Line
-	4275 3150 4275 4025
 Wire Wire Line
 	3650 2900 3650 2275
@@
 P 5200 3150
 F 0 "R301" H 5270 3196 50  0000 L CNN
-F 1 "10K" H 5270 3105 50  0000 L CNN
+F 1 "39K" H 5270 3105 50  0000 L CNN
 F 2 "Resistor_SMD:R_0805_2012Metric_Pad1.15x1.40mm_HandSolder" V 5130 3150 50  0001 C CNN
-F 3 "~" H 5200 3150 50  0001 C CNN
+F 3 "https://www.mouser.at/datasheet/2/427/crcwce3-1762584.pdf" H 5200 3150 50  0001 C CNN
+F 4 "CRCW040239K0FKEDC" H 5200 3150 50  0001 C CNN "MPN"
 	1    5200 3150
 	1    0    0    -1
@@
 P 5200 3750
 F 0 "R302" H 5270 3796 50  0000 L CNN
-F 1 "15K" H 5270 3705 50  0000 L CNN
+F 1 "27K" H 5270 3705 50  0000 L CNN
 F 2 "Resistor_SMD:R_0805_2012Metric_Pad1.15x1.40mm_HandSolder" V 5130 3750 50  0001 C CNN
-F 3 "~" H 5200 3750 50  0001 C CNN
+F 3 "https://www.mouser.at/datasheet/2/427/crcwce3-1762584.pdf" H 5200 3750 50  0001 C CNN
+F 4 "CRCW120627K0FKEAC" H 5200 3750 50  0001 C CNN "MPN"
 	1    5200 3750
 	1    0    0    -1
 $EndComp
-Text HLabel 8700 5775 2    50   Input ~ 0
+Text HLabel 8700 6175 2    50   Input ~ 0
 IN-
-Text HLabel 8700 4475 2    50   Input ~ 0
+Text HLabel 8700 5175 2    50   Input ~ 0
 IN+
 $Comp
@@
 	7375 3575 7175 3575
 $Comp
-L Device:R R303
+L Device:R R307
 U 1 1 5E60E589
-P 8125 4800
-F 0 "R303" H 8195 4846 50  0000 L CNN
-F 1 "9K" H 8195 4755 50  0000 L CNN
-F 2 "Resistor_SMD:R_0805_2012Metric_Pad1.15x1.40mm_HandSolder" V 8055 4800 50  0001 C CNN
-F 3 "~" H 8125 4800 50  0001 C CNN
-	1    8125 4800
-	1    0    0    -1
-$EndComp
-$Comp
-L Device:R R304
+P 8125 5425
+F 0 "R307" H 8195 5471 50  0000 L CNN
+F 1 "18K" H 8195 5380 50  0000 L CNN
+F 2 "Resistor_SMD:R_0805_2012Metric_Pad1.15x1.40mm_HandSolder" V 8055 5425 50  0001 C CNN
+F 3 "https://www.mouser.at/datasheet/2/418/NG_DS_9-1773463-9_A-1358566.pdf" H 8125 5425 50  0001 C CNN
+F 4 "CRGP0805F18K" H 8125 5425 50  0001 C CNN "MPN"
+	1    8125 5425
+	1    0    0    -1
+$EndComp
+$Comp
+L Device:R R308
 U 1 1 5E60E864
-P 8125 5475
-F 0 "R304" H 8195 5521 50  0000 L CNN
-F 1 "1K" H 8195 5430 50  0000 L CNN
-F 2 "Resistor_SMD:R_0805_2012Metric_Pad1.15x1.40mm_HandSolder" V 8055 5475 50  0001 C CNN
-F 3 "~" H 8125 5475 50  0001 C CNN
-	1    8125 5475
-	1    0    0    -1
-$EndComp
-Wire Wire Line
-	8125 5775 8125 5625
-Wire Wire Line
-	8125 5325 8125 5125
-Wire Wire Line
-	8125 5125 6175 5125
+P 8125 5925
+F 0 "R308" H 8195 5971 50  0000 L CNN
+F 1 "2K" H 8195 5880 50  0000 L CNN
+F 2 "Resistor_SMD:R_0805_2012Metric_Pad1.15x1.40mm_HandSolder" V 8055 5925 50  0001 C CNN
+F 3 "https://www.mouser.at/datasheet/2/427/crcwce3-1762584.pdf" H 8125 5925 50  0001 C CNN
+F 4 "CRCW08052K00FKEAC" H 8125 5925 50  0001 C CNN "MPN"
+	1    8125 5925
+	1    0    0    -1
+$EndComp
+Wire Wire Line
+	8125 5675 6175 5675
 Wire Wire Line
 	6175 3675 6575 3675
-Connection ~ 8125 5125
-Text Notes 8200 4450 0    50   ~ 0
+Text Notes 8200 5150 0    50   ~ 0
 0-20V
-Text Notes 7200 5100 0    50   ~ 0
+Text Notes 7200 5650 0    50   ~ 0
 0-2V
 Wire Wire Line
 	8700 3575 7775 3575
 Wire Wire Line
-	8125 5775 8700 5775
-Wire Wire Line
-	8125 4475 8700 4475
-Wire Wire Line
-	8125 4475 8125 4650
-Wire Wire Line
-	8125 4950 8125 5125
+	8125 6175 8700 6175
+Wire Wire Line
+	8125 5175 8700 5175
 Wire Wire Line
 	5200 3475 6575 3475
@@
 F 1 "0.1U" H 2390 2680 50  0000 L CNN
 F 2 "Capacitor_SMD:C_0805_2012Metric_Pad1.15x1.40mm_HandSolder" H 2313 2575 50  0001 C CNN
-F 3 "~" H 2275 2725 50  0001 C CNN
+F 3 "https://www.mouser.at/datasheet/2/445/885012207098-1727748.pdf" H 2275 2725 50  0001 C CNN
+F 4 "885012207098" H 2275 2725 50  0001 C CNN "MPN"
 	1    2275 2725
 	1    0    0    -1
@@
 Wire Wire Line
 	7675 3925 6175 3925
-Connection ~ 6175 3925
-Wire Wire Line
-	6175 3925 6175 5125
-Wire Wire Line
-	8375 4025 8375 4325
-Wire Wire Line
-	8375 4325 7550 4325
-Wire Wire Line
-	7550 4325 7550 4125
 Wire Wire Line
 	7550 4125 7675 4125
@@
 Wire Wire Line
 	8375 4025 8275 4025
+Wire Wire Line
+	8125 5575 8125 5675
+Connection ~ 8125 5675
+Wire Wire Line
+	8125 5675 8125 5775
+Wire Wire Line
+	8125 6175 8125 6075
+Wire Wire Line
+	8125 5275 8125 5175
+Wire Wire Line
+	6175 3925 6175 5675
+Connection ~ 6175 3925
+$Comp
+L Device:R R306
+U 1 1 5E7D0474
+P 7950 4475
+F 0 "R306" V 8157 4475 50  0000 C CNN
+F 1 "39K" V 8066 4475 50  0000 C CNN
+F 2 "Resistor_SMD:R_0805_2012Metric_Pad1.15x1.40mm_HandSolder" V 7880 4475 50  0001 C CNN
+F 3 "https://www.mouser.at/datasheet/2/427/crcwce3-1762584.pdf" H 7950 4475 50  0001 C CNN
+F 4 "CRCW040239K0FKEDC" H 7950 4475 50  0001 C CNN "MPN"
+	1    7950 4475
+	0    -1   -1   0
+$EndComp
+Wire Wire Line
+	8375 4475 8100 4475
+Wire Wire Line
+	8375 4025 8375 4475
+Wire Wire Line
+	7800 4475 7550 4475
+Wire Wire Line
+	7550 4125 7550 4475
+$Comp
+L Device:R R304
+U 1 1 5E7D2755
+P 7550 4725
+F 0 "R304" H 7620 4771 50  0000 L CNN
+F 1 "27K" H 7620 4680 50  0000 L CNN
+F 2 "Resistor_SMD:R_0805_2012Metric_Pad1.15x1.40mm_HandSolder" V 7480 4725 50  0001 C CNN
+F 3 "https://www.mouser.at/datasheet/2/427/crcwce3-1762584.pdf" H 7550 4725 50  0001 C CNN
+F 4 "CRCW120627K0FKEAC" H 7550 4725 50  0001 C CNN "MPN"
+	1    7550 4725
+	1    0    0    -1
+$EndComp
+Wire Wire Line
+	7550 4575 7550 4475
+Connection ~ 7550 4475
+$Comp
+L power:GND #PWR?
+U 1 1 5E7D3274
+P 7550 5325
+AR Path="/5E7D3274" Ref="#PWR?"  Part="1"
+AR Path="/5E5EBC79/5E7D3274" Ref="#PWR?"  Part="1"
+AR Path="/5E5EBE75/5E7D3274" Ref="#PWR0305"  Part="1"
+F 0 "#PWR0305" H 7550 5075 50  0001 C CNN
+F 1 "GND" H 7555 5152 50  0000 C CNN
+F 2 "" H 7550 5325 50  0001 C CNN
+F 3 "" H 7550 5325 50  0001 C CNN
+	1    7550 5325
+	1    0    0    -1
+$EndComp
+Text Notes 7925 4825 0    50   ~ 0
+Amplification of 1.65 here gives full range\nADC input for sense voltage range of 0-2V.
+$Comp
+L Device:R R303
+U 1 1 5E7FA900
+P 5200 4100
+F 0 "R303" H 5270 4146 50  0000 L CNN
+F 1 "33K" H 5270 4055 50  0000 L CNN
+F 2 "Resistor_SMD:R_0805_2012Metric_Pad1.15x1.40mm_HandSolder" V 5130 4100 50  0001 C CNN
+F 3 "https://www.mouser.at/datasheet/2/418/NG_DS_9-1773463-9_A-1358566.pdf" H 5200 4100 50  0001 C CNN
+F 4 "CRGP0805F33K" H 5200 4100 50  0001 C CNN "MPN"
+	1    5200 4100
+	1    0    0    -1
+$EndComp
+Wire Wire Line
+	5200 3950 5200 3900
+Wire Wire Line
+	5200 4250 5200 4325
+Wire Wire Line
+	4275 4325 5200 4325
+Wire Wire Line
+	4275 3150 4275 4325
+Connection ~ 5200 4325
+Wire Wire Line
+	5200 4325 5200 4400
+$Comp
+L Device:R R305
+U 1 1 5E7FE2C5
+P 7550 5100
+F 0 "R305" H 7620 5146 50  0000 L CNN
+F 1 "33K" H 7620 5055 50  0000 L CNN
+F 2 "Resistor_SMD:R_0805_2012Metric_Pad1.15x1.40mm_HandSolder" V 7480 5100 50  0001 C CNN
+F 3 "https://www.mouser.at/datasheet/2/418/NG_DS_9-1773463-9_A-1358566.pdf" H 7550 5100 50  0001 C CNN
+F 4 "CRGP0805F33K" H 7550 5100 50  0001 C CNN "MPN"
+	1    7550 5100
+	1    0    0    -1
+$EndComp
+Wire Wire Line
+	7550 4875 7550 4950
+Wire Wire Line
+	7550 5250 7550 5325
 $EndSCHEMATC

Commit message: Start of revision 2 design changes
Parts:
- removed D301: 1N914, Diode_SMD:D_SOD-123F, symbol pspice:DIODE
- removed U102: TLV4333, Package_SO:SOIC-14_3.9x8.7mm_P1.27mm, symbol teensy-load:TLV4333
- added C302, C303: 0.1U, Capacitor_SMD:C_0805_2012Metric_Pad1.15x1.40mm_HandSolder, symbol Device:C
- added D301: 1N914, Diode_SMD:D_SOD-123F, symbol Device:D
- added U302: LMV331, Package_TO_SOT_SMD:SOT-23-5, symbol Comparator:LMV331
- added U303: TLV333IDBVR, Package_TO_SOT_SMD:SOT-23-5, symbol teensy-load:TLV333IDBVR
Connections:
- net +3V3: now also C302.1, C303.1, U302.5 (V+), U303.5 (V+)
- net FET_GATE: now also D301.2 (A)
- net GND: now also C302.2, C303.2, U302.2 (V-), U303.2 (V-)
- net V_SENSE: now also U303.1
- net at R301.2, R302.1: now also U302.1 (+)
- net at R307.2, R308.1: now also U302.3 (-), U303.3 (+)
- net at R304.1, R306.1: now also U303.4 (-)
- new net: D301.1 (K), U302.4
Other:
- note added: "Amplification of 1.65\nhere gives full range\nADC input for sense\nvoltage range of 0-2V."
- note removed: "Amplification of 1.65 here gives full range\nADC input for sense voltage range of 0-2V."
- moved on the sheet: R304, R305, R306
